Commit message: fix: align simulator chassis frames with hardware geometry

File: src/duojin01_description/urdf/dual_arm_mobile.urdf (robot description, URDF)
Before this commit: robot dual_arm_mobile, 29 links, 28 joints
Links:
- added link laser
- link base_link: geometry collision box size=0.427 0.381 0.197; visual mesh filename=package://duojin01_description/models/dual_arm_mobile/meshe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
- link front_left_wheel: geometry collision cylinder length=0.0499999970198 radius=0.0503669815498; visual mesh filename=package://duojin01_description/models/dual_arm_mobile/meshe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
- link front_right_wheel: geometry collision cylinder length=0.0499999970198 radius=0.0503669874594; visual mesh filename=package://duojin01_description/models/dual_arm_mobile/meshe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
- link rear_left_wheel: geometry collision cylinder length=0.0499999970198 radius=0.050366981054; visual mesh filename=package://duojin01_description/models/dual_arm_mobile/meshe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
- link rear_right_wheel: geometry collision cylinder length=0.0499999970198 radius=0.0503669857583; visual mesh filename=package://duojin01_description/models/dual_arm_mobile/meshe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
Joints:
- added joint laser_frame_joint: type fixed, parent lidar_link, child laser, origin xyz=0 0 0 rpy=0 0 0
- joint front_left_wheel_joint: origin xyz=0.134954441 0.177700005 0.0513435919 rpy=0 0 0 -> xyz=0.15632214386 0.177691020072 0.0513076659357 rpy=0 0 0
- joint front_right_wheel_joint: origin xyz=0.135058369 -0.177682035 0.0542215877 rpy=0 0 0 -> xyz=0.156433566859 -0.177691020072 0.0542500428386 rpy=0 0 0
- joint lidar_link_joint: origin xyz=0.0618320881 3.32761556e-06 0.130232666 rpy=0 0 0 -> xyz=0.0924721442817 -8.97794961929e-06 0.130232665815 rpy=0 0 0
- joint lift_carriage_joint: origin xyz=0.0238344788 2.25061269e-08 0.692307662 rpy=0 0 0 -> xyz=0.0452233465265 -8.95544349239e-06 0.692307662 rpy=0 0 0
- joint rear_left_wheel_joint: origin xyz=-0.177814469 0.1774 0.0503129973 rpy=0 0 0 -> xyz=-0.156377854743 0.177391014993 0.0503076651713 rpy=0 0 0
- joint rear_right_wheel_joint: origin xyz=-0.177738957 -0.177382044 0.0502942237 rpy=0 0 0 -> xyz=-0.156377855977 -0.177391014993 0.0503076648392 rpy=0 0 0
