Commit message: Simplify maintenance structure and isolate regression workflows
Keep the current navigation/SLAM algorithms and numerical defaults unchanged.
Consolidate localization and keyboard defaults, derive online parameters from
the selected SLAM configuration, and repair map recovery/input boundaries.
Remove obsolete map synchronization, empty layouts and shaft frames; fix
shutdown lifecycle and verify offline tests with packaged backend source.

Validation: 124 Python tests, 12 launch argument checks, 14 CTest cases,
SLAM workflows and 40 command-chain checks passed in an isolated clean checkout.

File: src/duojin01_description/urdf/duojin01_hardware.xacro (robot description, xacro)
@@ -4,15 +4,8 @@
   <!-- Native CAD visuals use metres. Collision envelopes are independent. -->
   <xacro:macro name="mecanum_wheel_unit" params="prefix cad_name x y z radius width">
-    <!-- Preserve existing shaft/joint names at the measured axle, without fake shafts. -->
-    <joint name="${prefix}_wheel_shaft_joint" type="fixed">
+    <joint name="${prefix}_wheel_joint" type="continuous">
       <parent link="base_link" />
-      <child link="${prefix}_wheel_shaft" />
+      <child link="${prefix}_wheel" />
       <origin xyz="${x} ${y} ${z}" rpy="0 0 0" />
-    </joint>
-    <link name="${prefix}_wheel_shaft" />
-    <joint name="${prefix}_wheel_joint" type="continuous">
-      <parent link="${prefix}_wheel_shaft" />
-      <child link="${prefix}_wheel" />
-      <origin xyz="0 0 0" rpy="0 0 0" />
       <axis xyz="0 1 0" />
     </joint>
